Commit message: created the folder for the description

File: robot_simulation_description/urdf/ball.xacro (robot description, xacro)
@@ -1,5 +1,5 @@
 <?xml version="1.0"?>
 <robot xmlns:xacro="http://www.ros.org/wiki/xacro" name="ball">
-<xacro:include filename="$(find robot_simulation)/urdf/ball.gazebo"/>
+<xacro:include filename="$(find robot_simulation_description)/urdf/ball.gazebo"/>
   <material name="black">
     <color rgba="0.0 0.0 0.0 1.0"/>

File: robot_simulation_description/urdf/robot.xacro (robot description, xacro)
@@ -1,9 +1,7 @@
-<?xml version="1.0" ?>
-<robot name="robot_rot_camera" xmlns:xacro="http://ros.org/wiki/xacro">
-<xacro:include filename="$(find robot_simulation)/urdf/robot_rot_camera.gazebo"/>
-    <!--    Define weels properies  -->
+<?xml version="1.0"?>
+<robot xmlns:xacro="http://www.ros.org/wiki/xacro" name="robot_xacro">
+    <xacro:include filename="$(find robot_simulation_description)/urdf/robot.gazebo"/>
     <xacro:property name="length_wheel" value="0.04" />
     <xacro:property name="radius_wheel" value="0.1" />
-    <!--    Define a general inertial matrix    -->
     <xacro:macro name="default_inertial" params="mass">
         <inertial>
@@ -13,5 +11,4 @@
         </inertial>
     </xacro:macro>
-    <!--    Define the wheel geometry   -->
     <xacro:macro name="wheel_geometry">
         <geometry>
@@ -19,5 +16,4 @@
         </geometry>
     </xacro:macro>
-    <!--    Define a bunch of colors    -->
     <material name="black">
         <color rgba="0.0 0.0 0.0 1.0"/>
@@ -47,5 +43,5 @@
                                     THE LINKS
     ########################################################################### -->
-    <!--    Define the moving platform link -->
+    <!--    The moving platform -->
     <link name="link_chassis">
         <!-- pose and inertial -->
@@ -56,5 +52,5 @@
             <inertia ixx="0.0395416666667" ixy="0" ixz="0" iyy="0.106208333333" iyz="0" izz="0.106208333333"/>
         </inertial>
-        <!--    The body of the moving platform    -->
+        <!-- body -->
         <collision name="collision_chassis">
             <geometry>
@@ -69,7 +65,7 @@
             <material name="blue"/>
         </visual>
-        <!--    The castor wheel in the front  -->
+        <!-- caster front -->
         <collision name="caster_front_collision">
-            <origin rpy=" 0 0 0" xyz="0.2 0 -0.05"/>
+            <origin rpy=" 0 0 0" xyz="0.35 0 -0.05"/>
             <geometry>
                 <sphere radius="0.05"/>
@@ -83,5 +79,5 @@
         </visual>
     </link>
-    <!--    The fixed wheel on the right    -->
+    <!--    The right Wheel -->
     <link name="link_right_wheel">
         <xacro:default_inertial mass="0.2"/>
@@ -93,11 +89,11 @@
             <origin rpy="0 1.5707 1.5707" xyz="0 0 0"/>
             <xacro:wheel_geometry />
-            <material name="yellow"/>
+            <material name="red"/>
         </visual>
     </link>
-    <!--    The fixed wheel on the left -->
+    <!--    The left wheel  -->
     <link name="link_left_wheel">
         <xacro:default_inertial mass="0.2"/>
-        <collision name="link_lef_wheel_collision">
+        <collision name="link_left_wheel_collision">
             <origin rpy="0 1.5707 1.5707" xyz="0 0 0"/>
             <xacro:wheel_geometry />
@@ -109,6 +105,6 @@
         </visual>
     </link>
-    <!--    The rotating base where the camera is placed    -->
-    <link name="link_rotating_base">
+    <!--    The neck    -->
+    <link name="link_neck">
         <inertial>
             <mass value="0.1"/>
@@ -117,39 +113,45 @@
         </inertial>
         <collision name="link_rotating_base_collision">
-            <origin rpy="0 0 0" xyz="0 0 0" />
+            <origin rpy="0 0 0" xyz="0 0 0.05" />
             <geometry>
-                <cylinder length="0.50" radius="0.05"/>
+                <cylinder length="0.10" radius="0.05"/>
             </geometry>
         </collision>
         <visual name="link_rotating_base_visual" >
-            <origin rpy="0 0 0" xyz="0 0 0" />
+            <origin rpy="0 0 0" xyz="0 0 0.05" />
             <geometry>
-                <cylinder length="0.50" radius="0.05"/>
+                <cylinder length="0.10" radius="0.05"/>
             </geometry>
             <material name="green"/>
         </visual>
     </link>
-    <!--    The camera  -->
-    <link name="link_camera" >
-        <collision name="link_camera_collision">
-            <origin rpy="0 0 0" xyz="0 0 0" />
+    <!--    The Camera  -->
+    <link name="camera_link">
+        <collision>
+            <origin xyz="0 0 0.125" rpy="0 0 0"/>
             <geometry>
-                <box size="0.05 0.05 0.05"/>
+                <box size="0.2 0.2 0.2"/>
             </geometry>
         </collision>
-        <visual name="link_camera_visual" >
-            <origin rpy="0 0 0" xyz="0 0 0.025" />
+        <visual>
+            <origin xyz="0 0 0.1" rpy="0 0 0"/>
             <geometry>
-                <box size="0.05 0.05 0.05"/>
+                <box size="0.2 0.2 0.2"/>
             </geometry>
-            <material name="black"/>
+            <material name="brown">
+                <color rgba="1 0 0 1"/>
+            </material>
         </visual>
+        <inertial>
+            <mass value="1e-5" />
+            <origin xyz="0 0 0" rpy="0 0 0"/>
+            <inertia ixx="1e-6" ixy="0" ixz="0" iyy="1e-6" iyz="0" izz="1e-6" />
+        </inertial>
     </link>
 <!--###########################################################################
                                     THE JOINTS
     ########################################################################### -->
-    <!--    Joint form moving platform to right fixed wheel -->
     <joint name="joint_right_wheel" type="continuous">
-        <origin rpy="0 0 0" xyz="-0.05 -0.15 0"/>
+        <origin rpy="0 0 0" xyz="-0.05 0.15 0"/>
         <child link="link_right_wheel"/>
         <parent link="link_chassis"/>
@@ -158,7 +160,6 @@
         <joint_properties damping="1.0" friction="1.0"/>
     </joint>
-    <!--    Joint form moving platform to left fixed wheel -->
     <joint name="joint_left_wheel" type="continuous">
-        <origin rpy="0 0 0" xyz="-0.05 0.15 0"/>
+        <origin rpy="0 0 0" xyz="-0.05 -0.15 0"/>
         <child link="link_left_wheel"/>
         <parent link="link_chassis"/>
@@ -167,8 +168,8 @@
         <joint_properties damping="1.0" friction="1.0"/>
     </joint>
-    <!--    Joint form moving platform to to rotating base  -->
-    <joint name="joint_rotating_base" type="continuous">
-        <origin rpy="0 0 0" xyz="0 0 0.25"/>
-        <child link="link_rotating_base"/>
+    <!--    Joint form moving platform to the rotating base  -->
+    <joint name="joint_neck" type="continuous">
+        <origin rpy="0 0 0" xyz="0 0 0.035"/>
+        <child link="link_neck"/>
         <parent link="link_chassis"/>
         <axis rpy="0 0 0" xyz="0 0 1"/>
@@ -176,9 +177,20 @@
         <joint_properties damping="1.0" friction="1.0"/>
     </joint>
-    <!--    Joint form the rotating platfrom to the camera  -->
-    <joint name="joint_camera" type="fixed">
-        <origin xyz="0 0 0.25" rpy="0 0 0"/>
-        <parent link="link_rotating_base"/>
-        <child link="link_camera"/>
+    <!--    Joint form the neck to the camera  -->
+    <joint name="camera_joint" type="fixed">
+        <axis xyz="0 1 0" />
+        <origin xyz="0.0 0 0.05" rpy="0 0 0"/>
+        <parent link="link_neck"/>
+        <child link="camera_link"/>
     </joint>
+    <transmission name="neck_joint_transmission">
+        <type>transmission_interface/SimpleTransmission</type>
+        <joint name="joint_neck">
+            <hardwareInterface>hardware_interface/EffortJointInterface</hardwareInterface>
+        </joint>
+        <actuator name="motor_neck">
+            <hardwareInterface>hardware_interface/EffortJointInterface</hardwareInterface>
+            <mechanicalInterface>1</mechanicalInterface>
+        </actuator>
+    </transmission>
 </robot>

File: robot_simulation_description/urdf/robot_rot_camera.xacro (robot description, xacro)
@@ -1,7 +1,9 @@
-<?xml version="1.0"?>
-<robot xmlns:xacro="http://www.ros.org/wiki/xacro" name="robot_xacro">
-    <xacro:include filename="$(find robot_simulation)/urdf/robot.gazebo"/>
+<?xml version="1.0" ?>
+<robot name="robot_rot_camera" xmlns:xacro="http://ros.org/wiki/xacro">
+<xacro:include filename="$(find robot_simulation_description)/urdf/robot_rot_camera.gazebo"/>
+    <!--    Define weels properies  -->
     <xacro:property name="length_wheel" value="0.04" />
     <xacro:property name="radius_wheel" value="0.1" />
+    <!--    Define a general inertial matrix    -->
     <xacro:macro name="default_inertial" params="mass">
         <inertial>
@@ -11,4 +13,5 @@
         </inertial>
     </xacro:macro>
+    <!--    Define the wheel geometry   -->
     <xacro:macro name="wheel_geometry">
         <geometry>
@@ -16,4 +19,5 @@
         </geometry>
     </xacro:macro>
+    <!--    Define a bunch of colors    -->
     <material name="black">
         <color rgba="0.0 0.0 0.0 1.0"/>
@@ -43,5 +47,5 @@
                                     THE LINKS
     ########################################################################### -->
-    <!--    The moving platform -->
+    <!--    Define the moving platform link -->
     <link name="link_chassis">
         <!-- pose and inertial -->
@@ -52,5 +56,5 @@
             <inertia ixx="0.0395416666667" ixy="0" ixz="0" iyy="0.106208333333" iyz="0" izz="0.106208333333"/>
         </inertial>
-        <!-- body -->
+        <!--    The body of the moving platform    -->
         <collision name="collision_chassis">
             <geometry>
@@ -65,7 +69,7 @@
             <material name="blue"/>
         </visual>
-        <!-- caster front -->
+        <!--    The castor wheel in the front  -->
         <collision name="caster_front_collision">
-            <origin rpy=" 0 0 0" xyz="0.35 0 -0.05"/>
+            <origin rpy=" 0 0 0" xyz="0.2 0 -0.05"/>
             <geometry>
                 <sphere radius="0.05"/>
@@ -79,5 +83,5 @@
         </visual>
     </link>
-    <!--    The right Wheel -->
+    <!--    The fixed wheel on the right    -->
     <link name="link_right_wheel">
         <xacro:default_inertial mass="0.2"/>
@@ -89,11 +93,11 @@
             <origin rpy="0 1.5707 1.5707" xyz="0 0 0"/>
             <xacro:wheel_geometry />
-            <material name="red"/>
+            <material name="yellow"/>
         </visual>
     </link>
-    <!--    The left wheel  -->
+    <!--    The fixed wheel on the left -->
     <link name="link_left_wheel">
         <xacro:default_inertial mass="0.2"/>
-        <collision name="link_left_wheel_collision">
+        <collision name="link_lef_wheel_collision">
             <origin rpy="0 1.5707 1.5707" xyz="0 0 0"/>
             <xacro:wheel_geometry />
@@ -105,6 +109,6 @@
         </visual>
     </link>
-    <!--    The neck    -->
-    <link name="link_neck">
+    <!--    The rotating base where the camera is placed    -->
+    <link name="link_rotating_base">
         <inertial>
             <mass value="0.1"/>
@@ -113,45 +117,39 @@
         </inertial>
         <collision name="link_rotating_base_collision">
-            <origin rpy="0 0 0" xyz="0 0 0.05" />
+            <origin rpy="0 0 0" xyz="0 0 0" />
             <geometry>
-                <cylinder length="0.10" radius="0.05"/>
+                <cylinder length="0.50" radius="0.05"/>
             </geometry>
         </collision>
         <visual name="link_rotating_base_visual" >
-            <origin rpy="0 0 0" xyz="0 0 0.05" />
+            <origin rpy="0 0 0" xyz="0 0 0" />
             <geometry>
-                <cylinder length="0.10" radius="0.05"/>
+                <cylinder length="0.50" radius="0.05"/>
             </geometry>
             <material name="green"/>
         </visual>
     </link>
-    <!--    The Camera  -->
-    <link name="camera_link">
-        <collision>
-            <origin xyz="0 0 0.125" rpy="0 0 0"/>
+    <!--    The camera  -->
+    <link name="link_camera" >
+        <collision name="link_camera_collision">
+            <origin rpy="0 0 0" xyz="0 0 0" />
             <geometry>
-                <box size="0.2 0.2 0.2"/>
+                <box size="0.05 0.05 0.05"/>
             </geometry>
         </collision>
-        <visual>
-            <origin xyz="0 0 0.1" rpy="0 0 0"/>
+        <visual name="link_camera_visual" >
+            <origin rpy="0 0 0" xyz="0 0 0.025" />
             <geometry>
-                <box size="0.2 0.2 0.2"/>
+                <box size="0.05 0.05 0.05"/>
             </geometry>
-            <material name="brown">
-                <color rgba="1 0 0 1"/>
-            </material>
+            <material name="black"/>
         </visual>
-        <inertial>
-            <mass value="1e-5" />
-            <origin xyz="0 0 0" rpy="0 0 0"/>
-            <inertia ixx="1e-6" ixy="0" ixz="0" iyy="1e-6" iyz="0" izz="1e-6" />
-        </inertial>
     </link>
 <!--###########################################################################
                                     THE JOINTS
     ########################################################################### -->
+    <!--    Joint form moving platform to right fixed wheel -->
     <joint name="joint_right_wheel" type="continuous">
-        <origin rpy="0 0 0" xyz="-0.05 0.15 0"/>
+        <origin rpy="0 0 0" xyz="-0.05 -0.15 0"/>
         <child link="link_right_wheel"/>
         <parent link="link_chassis"/>
@@ -160,6 +158,7 @@
         <joint_properties damping="1.0" friction="1.0"/>
     </joint>
+    <!--    Joint form moving platform to left fixed wheel -->
     <joint name="joint_left_wheel" type="continuous">
-        <origin rpy="0 0 0" xyz="-0.05 -0.15 0"/>
+        <origin rpy="0 0 0" xyz="-0.05 0.15 0"/>
         <child link="link_left_wheel"/>
         <parent link="link_chassis"/>
@@ -168,8 +167,8 @@
         <joint_properties damping="1.0" friction="1.0"/>
     </joint>
-    <!--    Joint form moving platform to the rotating base  -->
-    <joint name="joint_neck" type="continuous">
-        <origin rpy="0 0 0" xyz="0 0 0.035"/>
-        <child link="link_neck"/>
+    <!--    Joint form moving platform to to rotating base  -->
+    <joint name="joint_rotating_base" type="continuous">
+        <origin rpy="0 0 0" xyz="0 0 0.25"/>
+        <child link="link_rotating_base"/>
         <parent link="link_chassis"/>
         <axis rpy="0 0 0" xyz="0 0 1"/>
@@ -177,20 +176,9 @@
         <joint_properties damping="1.0" friction="1.0"/>
     </joint>
-    <!--    Joint form the neck to the camera  -->
-    <joint name="camera_joint" type="fixed">
-        <axis xyz="0 1 0" />
-        <origin xyz="0.0 0 0.05" rpy="0 0 0"/>
-        <parent link="link_neck"/>
-        <child link="camera_link"/>
+    <!--    Joint form the rotating platfrom to the camera  -->
+    <joint name="joint_camera" type="fixed">
+        <origin xyz="0 0 0.25" rpy="0 0 0"/>
+        <parent link="link_rotating_base"/>
+        <child link="link_camera"/>
     </joint>
-    <transmission name="neck_joint_transmission">
-        <type>transmission_interface/SimpleTransmission</type>
-        <joint name="joint_neck">
-            <hardwareInterface>hardware_interface/EffortJointInterface</hardwareInterface>
-        </joint>
-        <actuator name="motor_neck">
-            <hardwareInterface>hardware_interface/EffortJointInterface</hardwareInterface>
-            <mechanicalInterface>1</mechanicalInterface>
-        </actuator>
-    </transmission>
 </robot>
