Commit message: moving on

File: robot_simulation_description/urdf/robot.xacro (robot description, xacro)
@@ -147,4 +147,26 @@
             <origin xyz="0 0 0" rpy="0 0 0"/>
             <inertia ixx="1e-6" ixy="0" ixz="0" iyy="1e-6" iyz="0" izz="1e-6" />
+        </inertial>
+    </link>
+    <link name="hokuyo_link">
+        <collision>
+          <origin xyz="0 0 0.025" rpy="0 0 0"/>
+          <geometry>
+      <box size="0.05 0.05 0.05"/>
+          </geometry>
+        </collision>
+        <visual>
+          <origin xyz="0 0 0.025" rpy="0 0 0"/>
+          <geometry>
+      <box size="0.05 0.05 0.05"/>
+          </geometry>
+          <material name="red">
+      <color rgba="1 0 0 1"/>
+          </material>
+        </visual>
+        <inertial>
+          <mass value="1e-5" />
+          <origin xyz="0 0 0" rpy="0 0 0"/>
+          <inertia ixx="1e-6" ixy="0" ixz="0" iyy="1e-6" iyz="0" izz="1e-6" />
         </inertial>
     </link>
@@ -194,3 +216,9 @@
         </actuator>
     </transmission>
+    <joint name="hokuyo_joint" type="fixed">
+        <axis xyz="0 1 0" />
+        <origin xyz="0.28 0 0.05" rpy="0 0 0"/>
+        <parent link="link_chassis"/>
+        <child link="hokuyo_link"/>
+   </joint>
 </robot>

Commit message: Auto stash before merge of "third_assignment" and "origin/third_assignment"

File: robot_simulation_description/urdf/robot.xacro (robot description, xacro)
@@ -151,4 +151,5 @@
     <link name="hokuyo_link">
         <collision>
+<<<<<<< Updated upstream
           <origin xyz="0 0 0.025" rpy="0 0 0"/>
           <geometry>
@@ -171,4 +172,26 @@
         </inertial>
     </link>
+=======
+        <origin xyz="0 0 0.025" rpy="0 0 0"/>
+            <geometry>
+                <box size="0.05 0.05 0.05"/>
+            </geometry>
+        </collision>
+        <visual>
+            <origin xyz="0 0 0.025" rpy="0 0 0"/>
+            <geometry>
+                <box size="0.05 0.05 0.05"/>
+            </geometry>
+            <material name="red">
+                <color rgba="1 0 0 1"/>
+            </material>
+        </visual>
+        <inertial>
+            <mass value="1e-5" />
+            <origin xyz="0 0 0" rpy="0 0 0"/>
+            <inertia ixx="1e-6" ixy="0" ixz="0" iyy="1e-6" iyz="0" izz="1e-6" />
+        </inertial>
+    </link>
+>>>>>>> Stashed changes
 <!--###########################################################################
                                     THE JOINTS
@@ -205,4 +228,10 @@
         <parent link="link_neck"/>
         <child link="camera_link"/>
+    </joint>
+    <joint name="hokuyo_joint" type="fixed">
+        <axis xyz="0 1 0" />
+        <origin xyz="0.28 0 0.05" rpy="0 0 0"/>
+        <parent link="link_chassis"/>
+        <child link="hokuyo_link"/>
     </joint>
     <transmission name="neck_joint_transmission">

Commit message: changed the robot for an optimal mapping

File: robot_simulation_description/urdf/robot.xacro (robot description, xacro)
@@ -151,5 +151,4 @@
     <link name="hokuyo_link">
         <collision>
-<<<<<<< Updated upstream
           <origin xyz="0 0 0.025" rpy="0 0 0"/>
           <geometry>
@@ -172,26 +171,4 @@
         </inertial>
     </link>
-=======
-        <origin xyz="0 0 0.025" rpy="0 0 0"/>
-            <geometry>
-                <box size="0.05 0.05 0.05"/>
-            </geometry>
-        </collision>
-        <visual>
-            <origin xyz="0 0 0.025" rpy="0 0 0"/>
-            <geometry>
-                <box size="0.05 0.05 0.05"/>
-            </geometry>
-            <material name="red">
-                <color rgba="1 0 0 1"/>
-            </material>
-        </visual>
-        <inertial>
-            <mass value="1e-5" />
-            <origin xyz="0 0 0" rpy="0 0 0"/>
-            <inertia ixx="1e-6" ixy="0" ixz="0" iyy="1e-6" iyz="0" izz="1e-6" />
-        </inertial>
-    </link>
->>>>>>> Stashed changes
 <!--###########################################################################
                                     THE JOINTS
@@ -214,15 +191,11 @@
     </joint>
     <!--    Joint form moving platform to the rotating base  -->
-    <joint name="joint_neck" type="continuous">
+    <joint name="joint_neck" type="fixed">
         <origin rpy="0 0 0" xyz="0 0 0.035"/>
         <child link="link_neck"/>
         <parent link="link_chassis"/>
-        <axis rpy="0 0 0" xyz="0 0 1"/>
-        <limit effort="10000" velocity="1000"/>
-        <joint_properties damping="1.0" friction="1.0"/>
     </joint>
     <!--    Joint form the neck to the camera  -->
     <joint name="camera_joint" type="fixed">
-        <axis xyz="0 1 0" />
         <origin xyz="0.0 0 0.05" rpy="0 0 0"/>
         <parent link="link_neck"/>
@@ -231,23 +204,7 @@
     <joint name="hokuyo_joint" type="fixed">
         <axis xyz="0 1 0" />
-        <origin xyz="0.28 0 0.05" rpy="0 0 0"/>
+        <origin xyz="0.28 0 0.025" rpy="0 0 0"/>
         <parent link="link_chassis"/>
         <child link="hokuyo_link"/>
     </joint>
-    <transmission name="neck_joint_transmission">
-        <type>transmission_interface/SimpleTransmission</type>
-        <joint name="joint_neck">
-            <hardwareInterface>hardware_interface/EffortJointInterface</hardwareInterface>
-        </joint>
-        <actuator name="motor_neck">
-            <hardwareInterface>hardware_interface/EffortJointInterface</hardwareInterface>
-            <mechanicalInterface>1</mechanicalInterface>
-        </actuator>
-    </transmission>
-    <joint name="hokuyo_joint" type="fixed">
-        <axis xyz="0 1 0" />
-        <origin xyz="0.28 0 0.05" rpy="0 0 0"/>
-        <parent link="link_chassis"/>
-        <child link="hokuyo_link"/>
-   </joint>
 </robot>

Commit message: improved robot shape

File: robot_simulation_description/urdf/robot.xacro (robot description, xacro)
@@ -55,5 +55,8 @@
         <collision name="collision_chassis">
             <geometry>
+                <cylinder length="0.07" radius="0.25"/>
+                <!--
                 <box size="0.5 0.3 0.07"/>
+                -->
             </geometry>
         </collision>
@@ -61,5 +64,8 @@
             <origin rpy="0 0 0" xyz="0 0 0"/>
             <geometry>
+                <cylinder length="0.07" radius="0.25"/>
+                <!--
                 <box size="0.5 0.3 0.07"/>
+                -->
             </geometry>
             <material name="blue"/>
@@ -113,15 +119,17 @@
         </inertial>
         <collision name="link_rotating_base_collision">
-            <origin rpy="0 0 0" xyz="0 0 0.05" />
-            <geometry>
-                <cylinder length="0.10" radius="0.05"/>
+            <origin rpy="0 0 0" xyz="0 0 0" />
+            <geometry>
+                <cylinder length="0.15" radius="0.05"/>
             </geometry>
         </collision>
         <visual name="link_rotating_base_visual" >
-            <origin rpy="0 0 0" xyz="0 0 0.05" />
-            <geometry>
-                <cylinder length="0.10" radius="0.05"/>
-            </geometry>
-            <material name="green"/>
+            <origin rpy="0 0 0" xyz="0 0 0" />
+            <geometry>
+                <cylinder length="0.15" radius="0.05"/>
+            </geometry>
+            <material name="green">
+              <color rgba="0 1 0 1"/>
+            </material>
         </visual>
     </link>
@@ -129,5 +137,5 @@
     <link name="camera_link">
         <collision>
-            <origin xyz="0 0 0.125" rpy="0 0 0"/>
+            <origin xyz="0 0 0" rpy="0 0 0"/>
             <geometry>
                 <box size="0.2 0.2 0.2"/>
@@ -135,5 +143,5 @@
         </collision>
         <visual>
-            <origin xyz="0 0 0.1" rpy="0 0 0"/>
+            <origin xyz="0 0 0" rpy="0 0 0"/>
             <geometry>
                 <box size="0.2 0.2 0.2"/>
@@ -162,5 +170,5 @@
           </geometry>
           <material name="red">
-      <color rgba="1 0 0 1"/>
+            <color rgba="1 0 0 1"/>
           </material>
         </visual>
@@ -192,5 +200,5 @@
     <!--    Joint form moving platform to the rotating base  -->
     <joint name="joint_neck" type="fixed">
-        <origin rpy="0 0 0" xyz="0 0 0.035"/>
+        <origin rpy="0 0 0" xyz="0 0 0.1"/>
         <child link="link_neck"/>
         <parent link="link_chassis"/>
@@ -198,5 +206,5 @@
     <!--    Joint form the neck to the camera  -->
     <joint name="camera_joint" type="fixed">
-        <origin xyz="0.0 0 0.05" rpy="0 0 0"/>
+        <origin xyz="0.0 0 0.175" rpy="0 0 0"/>
         <parent link="link_neck"/>
         <child link="camera_link"/>
@@ -204,5 +212,5 @@
     <joint name="hokuyo_joint" type="fixed">
         <axis xyz="0 1 0" />
-        <origin xyz="0.28 0 0.025" rpy="0 0 0"/>
+        <origin xyz="0.275 0 0.025" rpy="0 0 0"/>
         <parent link="link_chassis"/>
         <child link="hokuyo_link"/>

Commit message: update URDF

File: robot_simulation_description/urdf/robot.xacro (robot description, xacro)
@@ -71,7 +71,7 @@
             <material name="blue"/>
         </visual>
-        <!-- caster front -->
+        <!-- caster front
         <collision name="caster_front_collision">
-            <origin rpy=" 0 0 0" xyz="0.35 0 -0.05"/>
+            <origin rpy=" 0 0 0" xyz="0.2 0 -0.05"/>
             <geometry>
                 <sphere radius="0.05"/>
@@ -80,4 +80,68 @@
         <visual name="caster_front_visual">
             <origin rpy=" 0 0 0" xyz="0.2 0 -0.05"/>
+            <geometry>
+                <sphere radius="0.05"/>
+            </geometry>
+        </visual>-->
+    </link>
+    <!-- caster front  dummy-->
+    <link name="dummy_front_castor">
+            <xacro:default_inertial mass="0.001"/>
+        <collision name="link_dummy_front_castor_collision">
+            <origin rpy=" 0 0 0" xyz="0 0 0"/>
+            <geometry>
+                <sphere radius="0.05"/>
+            </geometry>
+        </collision>
+        <visual name="link_dummy_front_castor_visual">
+            <origin rpy=" 0 0 0" xyz="0 0 0"/>
+            <geometry>
+                <sphere radius="0.05"/>
+            </geometry>
+        </visual>
+    </link>
+    <!-- caster front -->
+    <link name="link_caster_front_wheel">
+            <xacro:default_inertial mass="0.2"/>
+        <collision name="link_caster_front_wheel_collision">
+            <origin rpy=" 0 0 0" xyz="0 0 0"/>
+            <geometry>
+                <sphere radius="0.05"/>
+            </geometry>
+        </collision>
+        <visual name="link_caster_front_wheel_visual">
+            <origin rpy=" 0 0 0" xyz="0 0 0"/>
+            <geometry>
+                <sphere radius="0.05"/>
+            </geometry>
+        </visual>
+    </link>
+    <!-- caster back  dummy-->
+    <link name="dummy_back_castor">
+            <xacro:default_inertial mass="0.001"/>
+        <collision name="link_dummy_back_castor_collision">
+            <origin rpy=" 0 0 0" xyz="0 0 0"/>
+            <geometry>
+                <sphere radius="0.05"/>
+            </geometry>
+        </collision>
+        <visual name="link_dummy_back_castor_visual">
+            <origin rpy=" 0 0 0" xyz="0 0 0"/>
+            <geometry>
+                <sphere radius="0.05"/>
+            </geometry>
+        </visual>
+    </link>
+    <!-- caster back -->
+    <link name="link_caster_back_wheel">
+            <xacro:default_inertial mass="0.2"/>
+        <collision name="link_caster_back_wheel_collision">
+            <origin rpy=" 0 0 0" xyz="0 0 0"/>
+            <geometry>
+                <sphere radius="0.05"/>
+            </geometry>
+        </collision>
+        <visual name="link_caster_back_wheel_visual">
+            <origin rpy=" 0 0 0" xyz="0 0 0"/>
             <geometry>
                 <sphere radius="0.05"/>
@@ -182,4 +246,36 @@
                                     THE JOINTS
     ########################################################################### -->
+    <joint name="joint_caster_back_dummy" type="continuous">
+        <origin rpy="0 0 0" xyz="-0.2 0 -0.05"/>
+        <child link="dummy_back_castor"/>
+        <parent link="link_chassis"/>
+        <axis rpy="0 0 0" xyz="1 0 0"/>
+        <limit effort="10000" velocity="1000"/>
+        <joint_properties damping="1.0" friction="1.0"/>
+    </joint>
+    <joint name="joint_caster_back_wheel" type="continuous">
+        <origin rpy="0 0 0" xyz="0 0 0"/>
+        <child link="link_caster_back_wheel"/>
+        <parent link="dummy_back_castor"/>
+        <axis rpy="0 0 0" xyz="0 1 0"/>
+        <limit effort="10000" velocity="1000"/>
+        <joint_properties damping="1.0" friction="1.0"/>
+    </joint>
+    <joint name="joint_caster_front_dummy" type="continuous">
+        <origin rpy="0 0 0" xyz="0.2 0 -0.05"/>
+        <child link="dummy_front_castor"/>
+        <parent link="link_chassis"/>
+        <axis rpy="0 0 0" xyz="1 0 0"/>
+        <limit effort="10000" velocity="1000"/>
+        <joint_properties damping="1.0" friction="1.0"/>
+    </joint>
+    <joint name="joint_caster_front_wheel" type="continuous">
+        <origin rpy="0 0 0" xyz="0 0 0"/>
+        <child link="link_caster_front_wheel"/>
+        <parent link="dummy_front_castor"/>
+        <axis rpy="0 0 0" xyz="0 1 0"/>
+        <limit effort="10000" velocity="1000"/>
+        <joint_properties damping="1.0" friction="1.0"/>
+    </joint>
     <joint name="joint_right_wheel" type="continuous">
         <origin rpy="0 0 0" xyz="-0.05 0.15 0"/>
